File: projects/8bit_pcb/OUT_7SEG.sch (EAGLE design)
At the start: 26 parts, among them IC4 74LS139N, IC5 NE555N

Commit message: RAM, Disp16Seg, Decoder
Parts:
- removed C1: (no value), rcl:CPOL-EUE3.5-8
- removed C7: (no value), rcl:C-EUC1206K
- added R10, R11, R12, R13, R14, R15, R16, R17, R41, R6, R7, R8, R9: 330, rcl:R-EU_R0805
- added R4: 1k, rcl:R-EU_0204/7
- added R5: 100k, rcl:R-EU_0204/7
- added U$10, U$9: CAP, IsaacAlonso:CAP
- C8: value (none) -> 10n; device rcl:C-EUC1206K -> rcl:CPOL-EUE2,5-6E
- R1, R2: value (none) -> 330; device rcl:R-EU_M1206 -> rcl:R-EU_R0805
- R3: value (none) -> 330; device rcl:R-TRIMM64W -> rcl:R-EU_R0805
Connections:
- removed net N$33: IC5.DIS, R1.2, R2.1
- removed net N$34: C8.1, IC5.CV
- new net ICLK: U$1.P33
- new net N$1: IC5.DIS, R4.1, R5.2
- new net N$10: EEPROM1G$1.I/O7, R9.1
- new net N$11: EEPROM0G$1.I/O0, R10.1
- new net N$12: EEPROM0G$1.I/O1, R11.1
- new net N$13: EEPROM0G$1.I/O2, R12.1
- new net N$14: EEPROM0G$1.I/O3, R13.1
- new net N$15: EEPROM0G$1.I/O4, R14.1
- new net N$16: EEPROM0G$1.I/O5, R16.1
- new net N$17: EEPROM0G$1.I/O6, R15.1
- new net N$18: EEPROM0G$1.I/O7, R17.1
- new net N$2: IC5.CV, U$9.P+
- new net N$3: EEPROM1G$1.I/O0, R41.1
- new net N$4: EEPROM1G$1.I/O1, R1.1
- new net N$6: EEPROM1G$1.I/O3, R3.1
- new net N$7: EEPROM1G$1.I/O4, R6.1
- new net N$8: EEPROM1G$1.I/O5, R7.1
- new net N$9: EEPROM1G$1.I/O6, R8.1
- net !WR_AUX: now also U$1.P17
- net !WR_OUTH: now also U$1.P23
- net !WR_OUTL: now also U$1.P22
- net BUS0: now also U$1.P2
- net BUS1: now also U$1.P37
- net BUS2: now also U$1.P3
- net BUS3: now also U$1.P36
- net BUS4: now also U$1.P4
- net BUS5: now also U$1.P35
- net BUS6: now also U$1.P5
- net BUS7: now also U$1.P34
- net CLK: now also U$1.P6
- net CLK2: now also CNTA.CLK
- net GND: now also C8.-, IC4B.A, IC4B.B, IC4B.G, U$1.P20, U$1.P21, U$10.P-, U$9.P-; no longer C1.-, C7.2, C8.2
- net N$36: now also R5.1, U$10.P+; no longer C7.1, R1.1
- net N$5: now also EEPROM1G$1.I/O2, R2.1; no longer U$1.P20, U$1.P21
- net OUT_0: now also R10.2; no longer EEPROM0G$1.I/O0
- net OUT_1: now also R11.2; no longer EEPROM0G$1.I/O1
- net OUT_10: now also R2.2; no longer EEPROM1G$1.I/O2
- net OUT_11: now also R3.2; no longer EEPROM1G$1.I/O3
- net OUT_12: now also R6.2; no longer EEPROM1G$1.I/O4
- net OUT_13: now also R7.2; no longer EEPROM1G$1.I/O5
- net OUT_14: now also R8.2; no longer EEPROM1G$1.I/O6
- net OUT_15: now also R9.2; no longer EEPROM1G$1.I/O7
- net OUT_2: now also R12.2; no longer EEPROM0G$1.I/O2
- net OUT_3: now also R13.2; no longer EEPROM0G$1.I/O3
- net OUT_4: now also R14.2; no longer EEPROM0G$1.I/O4
- net OUT_5: now also R16.2; no longer EEPROM0G$1.I/O5
- net OUT_6: now also R15.2; no longer EEPROM0G$1.I/O6
- net OUT_7: now also R17.2; no longer EEPROM0G$1.I/O7
- net OUT_8: now also R41.2; no longer EEPROM1G$1.I/O0
- net OUT_9: now also R1.2; no longer EEPROM1G$1.I/O1
- net RST: now also U$1.P7
- net VCC: now also C8.+, CNTA.CLR, CNTA.ENP, CNTA.ENT, CNTA.LD, R4.2; no longer C1.+, R2.2
Other:
- moved on the sheet: EEPROM1, U$2, U$3, U$4, U$5, U$6, U$7, U$8
